File: PCB Design/Microcontroller Schematics.kicad_sch (KiCad schematic)
At the start: 54 parts, among them J1 Power (9v), J10 Micro_SD_Card, J11 Throttle HallEffect, J12 Screen Connector, J13 Button 1, J14 Button 2, J15 Button 3, J16 Button 4, J17 Power OUT (9v), J18 Data (RX TX)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

Commit message: Remade the through hole (TH) PCB
Parts:
- removed C5: 100nF, symbol Device:C
- removed R18, R19: 10k, Resistor_THT:R_Axial_DIN0207_L6.3mm_D2.5mm_P10.16mm_Horizontal, symbol Device:R
- C1, C3, C4: footprint (none) -> Capacitor_THT:C_Disc_D5.1mm_W3.2mm_P5.00mm
- J1, J13, J14, J15, J16, J17, J18, J19, J2, J7, J8: footprint (none) -> Connector_JST:JST_EH_S2B-EH_1x02_P2.50mm_Horizontal
- J10: footprint (none) -> Connector_Card:microSD_HC_Hirose_DM3AT-SF-PEJM5
- J11, J21, J6, J9: footprint (none) -> Connector_JST:JST_EH_S3B-EH_1x03_P2.50mm_Horizontal
- J12, J20, J3: footprint (none) -> Connector_JST:JST_EH_S4B-EH_1x04_P2.50mm_Horizontal
- J4: value Conn_01x02_Socket -> Bat 1V; footprint (none) -> Connector_JST:JST_EH_S2B-EH_1x02_P2.50mm_Horizontal
- J5: value Conn_01x02_Socket -> Bat 1+2 V; footprint (none) -> Connector_JST:JST_EH_S2B-EH_1x02_P2.50mm_Horizontal
- R11, R12, R13, R15, R4, R5: footprint (none) -> Resistor_THT:R_Axial_DIN0207_L6.3mm_D2.5mm_P10.16mm_Horizontal
Connections:
- net SCL: now also U1.14 (D22)
- net SDA: now also U1.11 (D21)
- net at J6.2 (Pin_2): now also U1.23 (D25); no longer U1.14 (D22)
- net at U6.1 (3V3): now also J10.4 (VDD)
- net at U6.2 (GND), U6.29 (GND): now also J10.6 (VSS)
Other:
- note added: "Front System"
- note added: "Rear System"
- moved on the sheet: J10, J6
